Commit message: update robot parameter

File: robot/vito.urdf.xacro (robot description, xacro)
@@ -52,3 +52,23 @@
     <origin xyz="0.0 0.0 ${0.55 + 0.1}" rpy="0.0 0.0 3.141592"/>
   </xacro:kit_head>
+  <link name="left_hand_palm_ref_link">
+      <inertial>
+        <insert_block name="negligible_inertia"/>
+      </inertial>
+  </link>
+  <joint name="$left_hand_palm_ref_joint" type="fixed">
+    <origin xyz="0 0 0.07" rpy="${3.141592/2} 0 ${3.141592/2}"/>
+    <parent link="left_hand_palm_link" />
+    <child link="left_hand_palm_ref_link" />
+  </joint>
+    <link name="right_hand_palm_ref_link">
+      <inertial>
+        <insert_block name="negligible_inertia"/>
+      </inertial>
+  </link>
+  <joint name="$right_hand_palm_ref_joint" type="fixed">
+    <origin xyz="0 0 0.07" rpy="${3.141592/2} 0 ${3.141592/2}"/>
+    <parent link="right_hand_palm_link" />
+    <child link="right_hand_palm_ref_link" />
+  </joint>
 </robot>

Commit message: add a object remove

File: robot/vito.urdf.xacro (robot description, xacro)
@@ -17,5 +17,6 @@
                     height="0.910"
                     plate_thickness="0.05">
-    <origin xyz="-0.495 0.55 0" rpy="0 0 0"/>
+    <!-- <origin xyz="-0.495 0.55 0" rpy="0 0 0"/> -->
+    <origin xyz="-0.25 0.55 0" rpy="0 0 0"/>
   </xacro:model_table>
   <!-- WORKBENCH -->

Commit message: testing if vito can be controlled by torque usin hands

File: robot/vito.urdf.xacro (robot description, xacro)
@@ -8,5 +8,5 @@
   <xacro:include filename="$(find lwr_description)/model/kuka_lwr.urdf.xacro"/>
   <xacro:include filename="$(find soft_hand_description)/model/soft_hand.urdf.xacro"/>
-  <!-- <xacro:include filename="$(find kit_head_description)/model/kit_head.urdf.xacro"/> -->
+  <xacro:include filename="$(find kit_head_description)/model/kit_head.urdf.xacro"/>
   <link name="vito_anchor" />
   <!-- BODY -->
@@ -17,6 +17,5 @@
                     height="0.910"
                     plate_thickness="0.05">
-    <!-- <origin xyz="-0.495 0.55 0" rpy="0 0 0"/> -->
-    <origin xyz="-0.25 0.55 0" rpy="0 0 0"/>
+    <origin xyz="-0.495 0.55 0" rpy="0 0 0"/>
   </xacro:model_table>
   <!-- WORKBENCH -->
@@ -38,5 +37,5 @@
   </xacro:kuka_lwr>
   <!-- LEFT SOFTHAND -->
-  <xacro:soft_hand parent="left_arm_7_link" name="left_hand" left="true" withAdaptiveTransmission="true" useMimicTag="true">
+  <xacro:soft_hand parent="left_arm_7_link" name="left_hand" left="true" withAdaptiveTransmission="true" useMimicTag="$(arg use_mimic_tag)">
     <origin xyz="0 0 0" rpy="0 0 0"/>
   </xacro:soft_hand>
@@ -46,13 +45,12 @@
   </xacro:kuka_lwr>
   <!-- RIGHT SOFTHAND -->
-  <xacro:soft_hand parent="right_arm_7_link" name="right_hand" left="false" withAdaptiveTransmission="true" useMimicTag="true">
+  <xacro:soft_hand parent="right_arm_7_link" name="right_hand" left="false" withAdaptiveTransmission="true" useMimicTag="$(arg use_mimic_tag)">
     <origin xyz="0 0 0" rpy="0 0 0"/>
   </xacro:soft_hand>
   <!-- HEAD -->
-<!--   <xacro:kit_head name="head" parent="vito_anchor">
+  <xacro:kit_head name="head" parent="vito_anchor">
     <origin xyz="0.0 0.0 ${0.55 + 0.1}" rpy="0.0 0.0 3.141592"/>
   </xacro:kit_head>
- -->
-  <link name="left_hand_palm_ref_link">
+    <link name="left_hand_palm_ref_link">
       <inertial>
         <insert_block name="negligible_inertia"/>

Commit message: add some comments

File: robot/vito.urdf.xacro (robot description, xacro)
@@ -10,4 +10,9 @@
   <xacro:include filename="$(find kit_head_description)/model/kit_head.urdf.xacro"/>
   <link name="vito_anchor" />
+   <link name="world"/>
+  <joint name="fixed" type="fixed">
+    <parent link="world"/>
+    <child link="vito_anchor"/>
+  </joint>
   <!-- BODY -->
   <xacro:model_table name="table"
@@ -72,3 +77,8 @@
     <child link="right_hand_palm_ref_link" />
   </joint>
+    <gazebo reference=" ">
+      <!-- <gravity>0</gravity> -->
+      <turnGravityOff>true</turnGravityOff>
+      <!-- <material>Gazebo/Grey</material> -->
+    </gazebo>
 </robot>

Commit message: CAnceling gravity and flags for simulation or real

File: robot/vito.urdf.xacro (robot description, xacro)
@@ -54,7 +54,7 @@
   </xacro:soft_hand>
   <!-- HEAD -->
-  <xacro:kit_head name="head" parent="vito_anchor">
+<!--   <xacro:kit_head name="head" parent="vito_anchor">
     <origin xyz="0.0 0.0 ${0.55 + 0.1}" rpy="0.0 0.0 3.141592"/>
-  </xacro:kit_head>
+  </xacro:kit_head> -->
     <link name="left_hand_palm_ref_link">
       <inertial>
@@ -77,8 +77,3 @@
     <child link="right_hand_palm_ref_link" />
   </joint>
-    <gazebo reference=" ">
-      <!-- <gravity>0</gravity> -->
-      <turnGravityOff>true</turnGravityOff>
-      <!-- <material>Gazebo/Grey</material> -->
-    </gazebo>
 </robot>

Commit message: Reference hand coordinate system depend on the robot so we are soft hand independent for the Potential field controller

File: robot/vito.urdf.xacro (robot description, xacro)
@@ -57,23 +57,29 @@
     <origin xyz="0.0 0.0 ${0.55 + 0.1}" rpy="0.0 0.0 3.141592"/>
   </xacro:kit_head> -->
-    <link name="left_hand_palm_ref_link">
+  <link name="left_hand_palm_ref_link">
       <inertial>
         <insert_block name="negligible_inertia"/>
       </inertial>
   </link>
-  <joint name="$left_hand_palm_ref_joint" type="fixed">
-    <origin xyz="0 0 0.07" rpy="${3.141592/2} 0 ${3.141592/2}"/>
-    <parent link="left_hand_palm_link" />
+  <joint name="left_hand_palm_ref_joint" type="fixed">
+    <origin xyz="0.002 0.007 0.161" rpy="${3.141592/2} 0 ${3.141592/2}"/>
+    <parent link="left_arm_7_link" />
     <child link="left_hand_palm_ref_link" />
   </joint>
-    <link name="right_hand_palm_ref_link">
+  <gazebo reference="left_hand_palm_ref_link">
+    <gravity>true</gravity>
+  </gazebo>
+  <link name="right_hand_palm_ref_link">
       <inertial>
         <insert_block name="negligible_inertia"/>
       </inertial>
   </link>
-  <joint name="$right_hand_palm_ref_joint" type="fixed">
-    <origin xyz="0 0 0.07" rpy="${3.141592/2} 0 ${3.141592/2}"/>
-    <parent link="right_hand_palm_link" />
+  <joint name="right_hand_palm_ref_joint" type="fixed">
+    <origin xyz="0.002 -0.007 0.161" rpy="${3.141592/2} 0 ${3.141592/2}"/>
+    <parent link="right_arm_7_link" />
     <child link="right_hand_palm_ref_link" />
   </joint>
+  <gazebo reference="right_hand_palm_ref_link">
+    <gravity>true</gravity>
+  </gazebo>
 </robot>

Commit message: This code uses a branch different from kuka-lwr. Use with caution or ask Manuel Bonilla for know how

File: robot/vito.urdf.xacro (robot description, xacro)
@@ -63,5 +63,5 @@
   </link>
   <joint name="left_hand_palm_ref_joint" type="fixed">
-    <origin xyz="0.002 0.007 0.161" rpy="${3.141592/2} 0 ${3.141592/2}"/>
+    <origin xyz="0.010 0.007 0.192" rpy="${3.141592/2} 0 ${3.141592/2}"/>
     <parent link="left_arm_7_link" />
     <child link="left_hand_palm_ref_link" />
@@ -76,5 +76,5 @@
   </link>
   <joint name="right_hand_palm_ref_joint" type="fixed">
-    <origin xyz="0.002 -0.007 0.161" rpy="${3.141592/2} 0 ${3.141592/2}"/>
+    <origin xyz="0.010 0.000 0.192" rpy="${3.141592/2} 0 ${3.141592/2}"/>
     <parent link="right_arm_7_link" />
     <child link="right_hand_palm_ref_link" />

Commit message: Updating

File: robot/vito.urdf.xacro (robot description, xacro)
@@ -22,5 +22,5 @@
                     height="0.910"
                     plate_thickness="0.05">
-    <origin xyz="-0.495 0.55 0" rpy="0 0 0"/>
+    <origin xyz="-0.220 0.55 0" rpy="0 0 0"/>
   </xacro:model_table>
   <!-- WORKBENCH -->
